File: Board/MP1800_GOTEK.kicad_pcb (KiCad board)
At the start: 2 copper layers, 99.1 x 63.5 mm, 45 parts, among them J1 Conn_02x25_Top_Bottom, J2 Conn_02x17_Odd_Even, J3 Conn_02x04_Odd_Even, J5 Barrel_Jack_Switch, J6 Conn_01x04_Male, J7 Conn_01x04_Female, SW1 SW_SPDT, SW2 SW_SPDT, SW3 SW_SPDT, U1 74HC123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

Commit message: Revision 0.2.3
Routing:
- net GND: track 484.5 -> 486.2 mm
- net /+5V_IN: track 24.5 -> 25.0 mm
Other:
- board text added: "Rev. 0.2.3"
- board text removed: "Rev. 0.2.2"
